Commit message: Changes to make gripper build and spawn in Gazebo

File: onrobot_description/urdf/inc/rg_common.xacro (robot description, xacro)
@@ -152,12 +152,4 @@
     <xacro:inner_finger prefix="${prefix}" fingerprefix="${fingerprefix}"/>
   </xacro:macro>
-  <!-- Gazebo plugin macro (for ros2_control simulation) -->
-  <xacro:macro name="gazebo_plugin" params="prefix">
-    <gazebo>
-      <plugin filename="libgazebo_ros2_control.so" name="gazebo_ros2_control">
-        <!-- Add additional parameters as needed -->
-      </plugin>
-    </gazebo>
-  </xacro:macro>
   <!-- Simple transmission macro for a joint -->
   <xacro:macro name="transmission_macro" params="prefix joint_name">

File: onrobot_description/urdf/onrobot_macro.xacro (robot description, xacro)
@@ -5,7 +5,9 @@
         params="
         onrobot_type
+        namespace:=''
         prefix:=''
         sim_gazebo:=false
         use_fake_hardware:=false
+        control_yaml:='$(find onrobot_driver)/config/default_controllers.yaml'
         connection_type:=serial
         device:=/tmp/ttyUR
@@ -24,5 +26,11 @@
         <xacro:if value="${sim_gazebo}">
             <gazebo>
-                <plugin filename="libgazebo_ros2_control.so" name="gazebo_ros2_control"/>
+                <plugin filename="libgz_ros2_control-system.so"
+                    name="gz_ros2_control::GazeboSimROS2ControlPlugin">
+                    <parameters>${control_yaml}</parameters>
+                    <ros>
+                        <namespace>${namespace}</namespace>
+                    </ros>
+                </plugin>
             </gazebo>
         </xacro:if>
@@ -31,5 +39,5 @@
             <hardware>
                 <xacro:if value="${sim_gazebo}">
-                    <plugin>gazebo_ros2_control/GazeboSystem</plugin>
+                    <plugin>gz_ros2_control/GazeboSimSystem</plugin>
                 </xacro:if>
                 <xacro:if value="${use_fake_hardware}">

File: onrobot_description/urdf/rg2_macro.xacro (robot description, xacro)
@@ -30,5 +30,10 @@
   </xacro:macro>
   <xacro:macro name="finger_joint" params="prefix">
-    <link name="${prefix}finger_width_mock_link"/>
+    <link name="${prefix}finger_width_mock_link">
+      <inertial> <!-- Gazebo requires inertia, even if this isn't a physical link-->
+        <mass value="1.0E-6"/>
+        <inertia ixx="1.0E-6" ixy="1.0E-9" ixz="1.0E-9" iyy="1.0E-6" iyz="1.0E-9" izz="1.0E-6" />
+      </inertial>
+    </link>
     <joint name="${prefix}finger_width" type="prismatic">
       <origin xyz="0 0 0" rpy="0 0 0" />

File: onrobot_description/urdf/rg6_macro.xacro (robot description, xacro)
@@ -30,5 +30,10 @@
   </xacro:macro>
   <xacro:macro name="finger_joint" params="prefix">
-    <link name="${prefix}finger_width_mock_link"/>
+    <link name="${prefix}finger_width_mock_link">
+      <inertial> <!-- Gazebo requires inertia, even if this isn't a physical link-->
+        <mass value="1.0E-6"/>
+        <inertia ixx="1.0E-6" ixy="1.0E-9" ixz="1.0E-9" iyy="1.0E-6" iyz="1.0E-9" izz="1.0E-6" />
+      </inertial>
+    </link>
     <joint name="${prefix}finger_width" type="prismatic">
       <origin xyz="0 0 0" rpy="0 0 0" />
