Commit message: Update launch file to work with new URDFs

File: onrobot_description/urdf/rg2/rg2.description.xacro (robot description, xacro)
@@ -83,5 +83,5 @@
     <xacro:right_outer_knuckle_joint prefix="${prefix}" />
     <xacro:transmission_macro prefix="${prefix}" joint_name="finger_width" />
-    <joint name="${prefix}base_joint" type="fixed">
+    <joint name="${prefix}onrobot_base_joint" type="fixed">
       <xacro:insert_block name="origin" />
       <parent link="${parent}" />

File: onrobot_description/urdf/rg6/rg6.description.xacro (robot description, xacro)
@@ -83,5 +83,5 @@
     <xacro:right_outer_knuckle_joint prefix="${prefix}" />
     <xacro:transmission_macro prefix="${prefix}" joint_name="finger_width" />
-    <joint name="${prefix}base_joint" type="fixed">
+    <joint name="${prefix}onrobot_base_joint" type="fixed">
       <xacro:insert_block name="origin" />
       <parent link="${parent}" />
