Commit message: Reorganize URDFs for better use as subassemblies

File: onrobot_description/urdf/common/rg.description.xacro (robot description, xacro)
@@ -1,5 +1,6 @@
 <?xml version="1.0"?>
 <robot xmlns:xacro="http://www.ros.org/wiki/xacro">
-  <xacro:macro name="onrobot_base_link" params="prefix">
+  <!-- Common component macros -->
+  <xacro:macro name="onrobot_base_link" params="onrobot_type prefix">
     <xacro:if value="${onrobot_type == 'rg2'}">
       <xacro:property name="mass" value="0.78" />
@@ -38,14 +39,9 @@
         <origin xyz="0 0 0" rpy="0 0 0" />
         <geometry>
-          <mesh filename="package://onrobot_description/meshes/${onrobot_type}/collision/base_link.stl" />
+          <mesh
+            filename="package://onrobot_description/meshes/${onrobot_type}/collision/base_link.stl" />
         </geometry>
       </collision>
     </link>
-    <gazebo reference="${prefix}onrobot_base_link">
-      <mu1>1.0</mu1>
-      <mu2>1.0</mu2>
-      <selfCollide>false</selfCollide>
-      <material>Gazebo/White</material>
-    </gazebo>
   </xacro:macro>
   <xacro:macro name="outer_knuckle" params="prefix fingerprefix">
@@ -59,5 +55,6 @@
         <origin xyz="0 0 0" rpy="0 0 0" />
         <geometry>
-          <mesh filename="package://onrobot_description/meshes/${onrobot_type}/visual/outer_knuckle.stl" />
+          <mesh
+            filename="package://onrobot_description/meshes/${onrobot_type}/visual/outer_knuckle.stl" />
         </geometry>
         <material name="">
@@ -68,14 +65,9 @@
         <origin xyz="0 0 0" rpy="0 0 0" />
         <geometry>
-          <mesh filename="package://onrobot_description/meshes/${onrobot_type}/collision/outer_knuckle.stl" />
+          <mesh
+            filename="package://onrobot_description/meshes/${onrobot_type}/collision/outer_knuckle.stl" />
         </geometry>
       </collision>
     </link>
-    <gazebo reference="${prefix}${fingerprefix}_outer_knuckle">
-      <mu1>0.1</mu1>
-      <mu2>0.1</mu2>
-      <selfCollide>false</selfCollide>
-      <material>Gazebo/White</material>
-    </gazebo>
   </xacro:macro>
   <xacro:macro name="inner_knuckle" params="prefix fingerprefix">
@@ -89,5 +81,6 @@
         <origin xyz="0 0 0" rpy="0 0 0" />
         <geometry>
-          <mesh filename="package://onrobot_description/meshes/${onrobot_type}/visual/inner_knuckle.stl" />
+          <mesh
+            filename="package://onrobot_description/meshes/${onrobot_type}/visual/inner_knuckle.stl" />
         </geometry>
         <material name="">
@@ -98,14 +91,9 @@
         <origin xyz="0 0 0" rpy="0 0 0" />
         <geometry>
-          <mesh filename="package://onrobot_description/meshes/${onrobot_type}/collision/inner_knuckle.stl" />
+          <mesh
+            filename="package://onrobot_description/meshes/${onrobot_type}/collision/inner_knuckle.stl" />
         </geometry>
       </collision>
     </link>
-    <gazebo reference="${prefix}${fingerprefix}_inner_knuckle">
-      <mu1>0.1</mu1>
-      <mu2>0.1</mu2>
-      <selfCollide>false</selfCollide>
-      <material>Gazebo/White</material>
-    </gazebo>
   </xacro:macro>
   <xacro:macro name="inner_finger" params="prefix fingerprefix">
@@ -119,5 +107,6 @@
         <origin xyz="0 0 0" rpy="0 0 0" />
         <geometry>
-          <mesh filename="package://onrobot_description/meshes/${onrobot_type}/visual/inner_finger.stl" />
+          <mesh
+            filename="package://onrobot_description/meshes/${onrobot_type}/visual/inner_finger.stl" />
         </geometry>
         <material name="">
@@ -128,27 +117,19 @@
         <origin xyz="0 0 0" rpy="0 0 0" />
         <geometry>
-          <mesh filename="package://onrobot_description/meshes/${onrobot_type}/collision/inner_finger.stl" />
+          <mesh
+            filename="package://onrobot_description/meshes/${onrobot_type}/collision/inner_finger.stl" />
         </geometry>
       </collision>
     </link>
-    <gazebo reference="${prefix}${fingerprefix}_inner_finger">
-      <kp>1000000.0</kp>
-      <kd>1.0</kd>
-      <kd>1.0</kd>
-      <mu1>1.0</mu1>
-      <mu2>1.0</mu2>
-      <minDepth>0.00001</minDepth>
-      <selfCollide>false</selfCollide>
-      <material>Gazebo/Black</material>
-    </gazebo>
   </xacro:macro>
   <xacro:macro name="finger_joints" params="prefix fingerprefix reflect">
-    <xacro:inner_knuckle_joint prefix="${prefix}" fingerprefix="${fingerprefix}" reflect="${reflect}"/>
-    <xacro:inner_finger_joint prefix="${prefix}" fingerprefix="${fingerprefix}"/>
+    <xacro:inner_knuckle_joint prefix="${prefix}" fingerprefix="${fingerprefix}"
+      reflect="${reflect}" />
+    <xacro:inner_finger_joint prefix="${prefix}" fingerprefix="${fingerprefix}" />
   </xacro:macro>
   <xacro:macro name="finger_links" params="prefix fingerprefix">
-    <xacro:outer_knuckle prefix="${prefix}" fingerprefix="${fingerprefix}"/>
-    <xacro:inner_knuckle prefix="${prefix}" fingerprefix="${fingerprefix}"/>
-    <xacro:inner_finger prefix="${prefix}" fingerprefix="${fingerprefix}"/>
+    <xacro:outer_knuckle prefix="${prefix}" fingerprefix="${fingerprefix}" />
+    <xacro:inner_knuckle prefix="${prefix}" fingerprefix="${fingerprefix}" />
+    <xacro:inner_finger prefix="${prefix}" fingerprefix="${fingerprefix}" />
   </xacro:macro>
   <!-- Simple transmission macro for a joint -->

File: onrobot_description/urdf/rg2/rg2.description.xacro (robot description, xacro)
@@ -1,6 +1,7 @@
 <?xml version="1.0"?>
 <robot xmlns:xacro="http://ros.org/wiki/xacro">
-  <xacro:property name="onrobot_type" value="rg2" />
-  <xacro:include filename="$(find onrobot_description)/urdf/inc/rg_common.xacro" />
+  <!-- Include common macros -->
+  <xacro:include filename="$(find onrobot_description)/urdf/common/rg.macro.xacro" />
+  <!-- Define component macros -->
   <xacro:macro name="inner_knuckle_joint" params="prefix fingerprefix reflect">
     <joint name="${prefix}${fingerprefix}_inner_knuckle_joint" type="revolute">
@@ -32,5 +33,5 @@
     <link name="${prefix}finger_width_mock_link">
       <inertial> <!-- Gazebo requires inertia, even if this isn't a physical link-->
-        <mass value="1.0E-6"/>
+        <mass value="1.0E-6" />
         <inertia ixx="1.0E-6" ixy="1.0E-9" ixz="1.0E-9" iyy="1.0E-6" iyz="1.0E-9" izz="1.0E-6" />
       </inertial>
@@ -49,7 +50,8 @@
       <axis xyz="-1 0 0" />
       <limit lower="-0.558505" upper="0.785398" velocity="100.0" effort="1000" />
-      <mimic joint="${prefix}finger_width" multiplier="${0.85 * ((-0.558505 - 0.785398) / 0.110)}" offset="0.785398" />
+      <mimic joint="${prefix}finger_width" multiplier="${0.85 * ((-0.558505 - 0.785398) / 0.110)}"
+        offset="0.785398" />
     </joint>
-    <xacro:finger_joints prefix="${prefix}" fingerprefix="left" reflect="1.0"/>
+    <xacro:finger_joints prefix="${prefix}" fingerprefix="left" reflect="1.0" />
   </xacro:macro>
   <xacro:macro name="right_outer_knuckle_joint" params="prefix">
@@ -62,19 +64,28 @@
       <mimic joint="${prefix}finger_joint" multiplier="-1" offset="0" />
     </joint>
-    <xacro:finger_joints prefix="${prefix}" fingerprefix="right" reflect="-1.0"/>
+    <xacro:finger_joints prefix="${prefix}" fingerprefix="right" reflect="-1.0" />
   </xacro:macro>
-  <link name="${prefix}gripper_tcp" />
-  <joint name="${prefix}tcp_joint" type="fixed">
-    <origin xyz="0 0 0.218" rpy="0 0 0" />
-    <parent link="${prefix}onrobot_base_link" />
-    <child link="${prefix}gripper_tcp" />
-  </joint>
-  <xacro:macro name="onrobot_rg2" params="prefix">
-    <xacro:onrobot_base_link prefix="${prefix}" />
-    <xacro:finger_links prefix="${prefix}" fingerprefix="left"/>
-    <xacro:finger_links prefix="${prefix}" fingerprefix="right"/>
-    <xacro:finger_joint prefix="${prefix}"/>
-    <xacro:right_outer_knuckle_joint prefix="${prefix}"/>
-    <xacro:transmission_macro prefix="${prefix}" joint_name="finger_width"/>
+  <xacro:macro name="gripper_tcp" params="prefix">
+    <link name="${prefix}gripper_tcp" />
+    <joint name="${prefix}tcp_joint" type="fixed">
+      <origin xyz="0 0 0.218" rpy="0 0 0" />
+      <parent link="${prefix}onrobot_base_link" />
+      <child link="${prefix}gripper_tcp" />
+    </joint>
+  </xacro:macro>
+  <!-- Main description macro -->
+  <xacro:macro name="rg2_description" params="prefix parent *origin">
+    <xacro:onrobot_base_link onrobot_type="rg2" prefix="${prefix}" />
+    <xacro:finger_links onrobot_type="rg2" prefix="${prefix}" fingerprefix="left" />
+    <xacro:finger_links onrobot_type="rg2" prefix="${prefix}" fingerprefix="right" />
+    <xacro:finger_joint prefix="${prefix}" />
+    <xacro:gripper_tcp prefix="${prefix}" />
+    <xacro:right_outer_knuckle_joint prefix="${prefix}" />
+    <xacro:transmission_macro prefix="${prefix}" joint_name="finger_width" />
+    <joint name="${prefix}base_joint" type="fixed">
+      <xacro:insert_block name="origin" />
+      <parent link="${parent}" />
+      <child link="${prefix}onrobot_base_link" />
+    </joint>
   </xacro:macro>
 </robot>

File: onrobot_description/urdf/rg6/rg6.description.xacro (robot description, xacro)
@@ -1,6 +1,7 @@
 <?xml version="1.0"?>
 <robot xmlns:xacro="http://ros.org/wiki/xacro">
-  <xacro:property name="onrobot_type" value="rg6" />
-  <xacro:include filename="$(find onrobot_description)/urdf/inc/rg_common.xacro" />
+  <!-- Include common macros -->
+  <xacro:include filename="$(find onrobot_description)/urdf/common/rg.macro.xacro" />
+  <!-- Define component macros -->
   <xacro:macro name="inner_knuckle_joint" params="prefix fingerprefix reflect">
     <joint name="${prefix}${fingerprefix}_inner_knuckle_joint" type="revolute">
@@ -22,5 +23,5 @@
       <mimic joint="${prefix}finger_joint" multiplier="1" offset="0" />
     </joint>
-    <link name="${prefix}${fingerprefix}_finger_tip"/>
+    <link name="${prefix}${fingerprefix}_finger_tip" />
     <joint name="${prefix}${fingerprefix}_finger_tip_joint" type="fixed">
       <origin xyz="0 0.025 0.052" rpy="0 0 0" />
@@ -32,5 +33,5 @@
     <link name="${prefix}finger_width_mock_link">
       <inertial> <!-- Gazebo requires inertia, even if this isn't a physical link-->
-        <mass value="1.0E-6"/>
+        <mass value="1.0E-6" />
         <inertia ixx="1.0E-6" ixy="1.0E-9" ixz="1.0E-9" iyy="1.0E-6" iyz="1.0E-9" izz="1.0E-6" />
       </inertial>
@@ -49,7 +50,8 @@
       <axis xyz="-1 0 0" />
       <limit lower="-0.628319" upper="0.628319" velocity="2.0" effort="1000" />
-      <mimic joint="${prefix}finger_width" multiplier="${0.88 * ((-0.628319 - 0.628319) / 0.160)}" offset="0.628319" />
+      <mimic joint="${prefix}finger_width" multiplier="${0.88 * ((-0.628319 - 0.628319) / 0.160)}"
+        offset="0.628319" />
     </joint>
-    <xacro:finger_joints prefix="${prefix}" fingerprefix="left" reflect="1.0"/>
+    <xacro:finger_joints prefix="${prefix}" fingerprefix="left" reflect="1.0" />
   </xacro:macro>
   <xacro:macro name="right_outer_knuckle_joint" params="prefix">
@@ -62,19 +64,28 @@
       <mimic joint="${prefix}finger_joint" multiplier="-1" offset="0" />
     </joint>
-    <xacro:finger_joints prefix="${prefix}" fingerprefix="right" reflect="-1.0"/>
+    <xacro:finger_joints prefix="${prefix}" fingerprefix="right" reflect="-1.0" />
   </xacro:macro>
-  <link name="${prefix}gripper_tcp"/>
-  <joint name="${prefix}tcp_joint" type="fixed">
-    <origin xyz="0 0 0.268" rpy="0 0 0" />
-    <parent link="${prefix}onrobot_base_link" />
-    <child link="${prefix}gripper_tcp" />
-  </joint>
-  <xacro:macro name="onrobot_rg6" params="prefix">
-    <xacro:onrobot_base_link prefix="${prefix}" />
-    <xacro:finger_links prefix="${prefix}" fingerprefix="left"/>
-    <xacro:finger_links prefix="${prefix}" fingerprefix="right"/>
-    <xacro:finger_joint prefix="${prefix}"/>
-    <xacro:right_outer_knuckle_joint prefix="${prefix}"/>
-    <xacro:transmission_macro prefix="${prefix}" joint_name="finger_width"/>
+  <xacro:macro name="gripper_tcp" params="prefix">
+    <link name="${prefix}gripper_tcp" />
+    <joint name="${prefix}tcp_joint" type="fixed">
+      <origin xyz="0 0 0.268" rpy="0 0 0" />
+      <parent link="${prefix}onrobot_base_link" />
+      <child link="${prefix}gripper_tcp" />
+    </joint>
+  </xacro:macro>
+  <!-- Main description macro -->
+  <xacro:macro name="rg6_description" params="prefix parent *origin">
+    <xacro:onrobot_base_link onrobot_type="rg6" prefix="${prefix}" />
+    <xacro:finger_links onrobot_type="rg6" prefix="${prefix}" fingerprefix="left" />
+    <xacro:finger_links onrobot_type="rg6" prefix="${prefix}" fingerprefix="right" />
+    <xacro:finger_joint prefix="${prefix}" />
+    <xacro:gripper_tcp prefix="${prefix}" />
+    <xacro:right_outer_knuckle_joint prefix="${prefix}" />
+    <xacro:transmission_macro prefix="${prefix}" joint_name="finger_width" />
+    <joint name="${prefix}base_joint" type="fixed">
+      <xacro:insert_block name="origin" />
+      <parent link="${parent}" />
+      <child link="${prefix}onrobot_base_link" />
+    </joint>
   </xacro:macro>
 </robot>

Commit message: Remove redundant macro file

File: onrobot_description/urdf/common/rg.description.xacro (robot description, xacro)
@@ -45,5 +45,5 @@
     </link>
   </xacro:macro>
-  <xacro:macro name="outer_knuckle" params="prefix fingerprefix">
+  <xacro:macro name="outer_knuckle" params="onrobot_type prefix fingerprefix">
     <link name="${prefix}${fingerprefix}_outer_knuckle">
       <inertial>
@@ -71,5 +71,5 @@
     </link>
   </xacro:macro>
-  <xacro:macro name="inner_knuckle" params="prefix fingerprefix">
+  <xacro:macro name="inner_knuckle" params="onrobot_type prefix fingerprefix">
     <link name="${prefix}${fingerprefix}_inner_knuckle">
       <inertial>
@@ -97,5 +97,5 @@
     </link>
   </xacro:macro>
-  <xacro:macro name="inner_finger" params="prefix fingerprefix">
+  <xacro:macro name="inner_finger" params="onrobot_type prefix fingerprefix">
     <link name="${prefix}${fingerprefix}_inner_finger">
       <inertial>
@@ -128,8 +128,11 @@
     <xacro:inner_finger_joint prefix="${prefix}" fingerprefix="${fingerprefix}" />
   </xacro:macro>
-  <xacro:macro name="finger_links" params="prefix fingerprefix">
-    <xacro:outer_knuckle prefix="${prefix}" fingerprefix="${fingerprefix}" />
-    <xacro:inner_knuckle prefix="${prefix}" fingerprefix="${fingerprefix}" />
-    <xacro:inner_finger prefix="${prefix}" fingerprefix="${fingerprefix}" />
+  <xacro:macro name="finger_links" params="onrobot_type prefix fingerprefix">
+    <xacro:outer_knuckle onrobot_type="${onrobot_type}" prefix="${prefix}"
+      fingerprefix="${fingerprefix}" />
+    <xacro:inner_knuckle onrobot_type="${onrobot_type}" prefix="${prefix}"
+      fingerprefix="${fingerprefix}" />
+    <xacro:inner_finger onrobot_type="${onrobot_type}" prefix="${prefix}"
+      fingerprefix="${fingerprefix}" />
   </xacro:macro>
   <!-- Simple transmission macro for a joint -->

File: onrobot_description/urdf/rg2/rg2.description.xacro (robot description, xacro)
@@ -2,5 +2,5 @@
 <robot xmlns:xacro="http://ros.org/wiki/xacro">
   <!-- Include common macros -->
-  <xacro:include filename="$(find onrobot_description)/urdf/common/rg.macro.xacro" />
+  <xacro:include filename="$(find onrobot_description)/urdf/common/rg.description.xacro" />
   <!-- Define component macros -->
   <xacro:macro name="inner_knuckle_joint" params="prefix fingerprefix reflect">

File: onrobot_description/urdf/rg6/rg6.description.xacro (robot description, xacro)
@@ -2,5 +2,5 @@
 <robot xmlns:xacro="http://ros.org/wiki/xacro">
   <!-- Include common macros -->
-  <xacro:include filename="$(find onrobot_description)/urdf/common/rg.macro.xacro" />
+  <xacro:include filename="$(find onrobot_description)/urdf/common/rg.description.xacro" />
   <!-- Define component macros -->
   <xacro:macro name="inner_knuckle_joint" params="prefix fingerprefix reflect">

Commit message: Set off-axis inertias to zero, as this is more realistic and prevents phsyics simulation issues

File: onrobot_description/urdf/common/rg.description.xacro (robot description, xacro)
@@ -6,8 +6,8 @@
       <xacro:property name="mass" value="0.78" />
       <xacro:property name="ixx" value="1.0E-03" />
-      <xacro:property name="ixy" value="1.0E-06" />
-      <xacro:property name="ixz" value="1.0E-06" />
+      <xacro:property name="ixy" value="0" />
+      <xacro:property name="ixz" value="0" />
       <xacro:property name="iyy" value="1.0E-03" />
-      <xacro:property name="iyz" value="1.0E-06" />
+      <xacro:property name="iyz" value="0" />
       <xacro:property name="izz" value="1.0E-03" />
     </xacro:if>
@@ -15,8 +15,8 @@
       <xacro:property name="mass" value="1.25" />
       <xacro:property name="ixx" value="1.0E-03" />
-      <xacro:property name="ixy" value="1.0E-06" />
-      <xacro:property name="ixz" value="1.0E-06" />
+      <xacro:property name="ixy" value="0" />
+      <xacro:property name="ixz" value="0" />
       <xacro:property name="iyy" value="1.0E-03" />
-      <xacro:property name="iyz" value="1.0E-06" />
+      <xacro:property name="iyz" value="0" />
       <xacro:property name="izz" value="1.0E-03" />
     </xacro:if>
@@ -50,5 +50,5 @@
         <origin xyz="0.0 0.0 0.0" rpy="0 0 0" />
         <mass value="0.05" />
-        <inertia ixx="1.0E-03" ixy="1.0E-06" ixz="1.0E-06" iyy="1.0E-03" iyz="1.0E-06" izz="1.0E-03" />
+        <inertia ixx="1.0E-03" ixy="0" ixz="0" iyy="1.0E-03" iyz="0" izz="1.0E-03" />
       </inertial>
       <visual>
@@ -76,5 +76,5 @@
         <origin xyz="0.0 0.0 0.0" rpy="0 0 0" />
         <mass value="0.05" />
-        <inertia ixx="1.0E-03" ixy="1.0E-06" ixz="1.0E-06" iyy="1.0E-03" iyz="1.0E-06" izz="1.0E-03" />
+        <inertia ixx="1.0E-03" ixy="0" ixz="0" iyy="1.0E-03" iyz="0" izz="1.0E-03" />
       </inertial>
       <visual>
@@ -102,5 +102,5 @@
         <origin xyz="0.0 0.0 0.0" rpy="0 0 0" />
         <mass value="0.05" />
-        <inertia ixx="1.0E-03" ixy="1.0E-06" ixz="1.0E-06" iyy="1.0E-03" iyz="1.0E-06" izz="1.0E-03" />
+        <inertia ixx="1.0E-03" ixy="0" ixz="0" iyy="1.0E-03" iyz="0" izz="1.0E-03" />
       </inertial>
       <visual>

File: onrobot_description/urdf/rg2/rg2.description.xacro (robot description, xacro)
@@ -34,5 +34,5 @@
       <inertial> <!-- Gazebo requires inertia, even if this isn't a physical link-->
         <mass value="1.0E-6" />
-        <inertia ixx="1.0E-6" ixy="1.0E-9" ixz="1.0E-9" iyy="1.0E-6" iyz="1.0E-9" izz="1.0E-6" />
+        <inertia ixx="1.0E-6" ixy="0" ixz="0" iyy="1.0E-6" iyz="0" izz="1.0E-6" />
       </inertial>
     </link>

File: onrobot_description/urdf/rg6/rg6.description.xacro (robot description, xacro)
@@ -34,5 +34,5 @@
       <inertial> <!-- Gazebo requires inertia, even if this isn't a physical link-->
         <mass value="1.0E-6" />
-        <inertia ixx="1.0E-6" ixy="1.0E-9" ixz="1.0E-9" iyy="1.0E-6" iyz="1.0E-9" izz="1.0E-6" />
+        <inertia ixx="1.0E-6" ixy="0" ixz="0" iyy="1.0E-6" iyz="0" izz="1.0E-6" />
       </inertial>
     </link>
